Commit message: fixed icub_with_hands model

File: icub_with_hands/urdf/iCub.urdf (robot description, URDF)
Before this commit: robot ICub, 94 links, 93 joints
Links:
- link base_link: mass None -> 0.111
- link il0: mass None -> 0.111; geometry visual mesh filename=package://icub_with_hands/meshes/il0.dae
- link il1: mass None -> 0.111; geometry visual mesh filename=package://icub_with_hands/meshes/il1.dae
- link il2: mass None -> 0.111; geometry visual mesh filename=package://icub_with_hands/meshes/il2.dae
- link il3: mass None -> 0.111; geometry visual mesh filename=package://icub_with_hands/meshes/il3.dae
- link indexbase: mass None -> 0.111; geometry visual mesh filename=package://icub_with_hands/meshes/indexbase.dae
- link l0: mass None -> 0.111; geometry visual mesh filename=package://icub_with_hands/meshes/l0.dae
- link l1: mass None -> 0.111; geometry visual mesh filename=package://icub_with_hands/meshes/l1.dae
- link l2: mass None -> 0.111; geometry visual mesh filename=package://icub_with_hands/meshes/l2.dae
- link l3: mass None -> 0.111; geometry visual mesh filename=package://icub_with_hands/meshes/l3.dae
- link l4: mass None -> 0.111; geometry visual mesh filename=package://icub_with_hands/meshes/l4.dae
- link l5: mass None -> 0.111; geometry visual mesh filename=package://icub_with_hands/meshes/l5.dae
- link l6: mass None -> 0.111; geometry visual mesh filename=package://icub_with_hands/meshes/l6.dae
- link l7: mass None -> 0.111
- link l7s: mass None -> 0.111
- link l8: mass None -> 0.111; geometry visual mesh filename=package://icub_with_hands/meshes/l8.dae
- link l8s: mass None -> 0.111; geometry visual mesh filename=package://icub_with_hands/meshes/l8.dae
- link la0: mass None -> 0.111; geometry visual mesh filename=package://icub_with_hands/meshes/la0.dae
- link la1: mass None -> 0.111; geometry visual mesh filename=package://icub_with_hands/meshes/la1.dae
- link la2: mass None -> 0.111; geometry visual mesh filename=package://icub_with_hands/meshes/la2.dae
- link la3: mass None -> 0.111; geometry visual mesh filename=package://icub_with_hands/meshes/la3.dae
- link la4: mass None -> 0.111; geometry visual mesh filename=package://icub_with_hands/meshes/la4.dae
- link la5: mass None -> 0.111; geometry visual mesh filename=package://icub_with_hands/meshes/la5.dae
- link la6: mass None -> 0.111; geometry visual mesh filename=package://icub_with_hands/meshes/la6.dae
- link lail0: mass None -> 0.111; geometry visual mesh filename=package://icub_with_hands/meshes/lail0.dae
- link lail1: mass None -> 0.111; geometry visual mesh filename=package://icub_with_hands/meshes/lail1.dae
- link lail2: mass None -> 0.111; geometry visual mesh filename=package://icub_with_hands/meshes/lail2.dae
- link lail3: mass None -> 0.111; geometry visual mesh filename=package://icub_with_hands/meshes/lail3.dae
- link left_palm: mass None -> 0.111; geometry visual mesh filename=package://icub_with_hands/meshes/left_palm.dae
- link lil0: mass None -> 0.111; geometry visual mesh filename=package://icub_with_hands/meshes/lil0.dae
- link lil1: mass None -> 0.111; geometry visual mesh filename=package://icub_with_hands/meshes/lil1.dae
- link lil2: mass None -> 0.111; geometry visual mesh filename=package://icub_with_hands/meshes/lil2.dae
- link lil3: mass None -> 0.111; geometry visual mesh filename=package://icub_with_hands/meshes/lil3.dae
- link lindexbase: mass None -> 0.111; geometry visual mesh filename=package://icub_with_hands/meshes/lindexbase.dae
- link littlebase: mass None -> 0.111; geometry visual mesh filename=package://icub_with_hands/meshes/littlebase.dae
- link ll0: mass None -> 0.111; geometry visual mesh filename=package://icub_with_hands/meshes/ll0.dae
- link ll1: mass None -> 0.111; geometry visual mesh filename=package://icub_with_hands/meshes/ll1.dae
- link ll2: mass None -> 0.111; geometry visual mesh filename=package://icub_with_hands/meshes/ll2.dae
- link ll3: mass None -> 0.111; geometry visual mesh filename=package://icub_with_hands/meshes/ll3.dae
- link ll4: mass None -> 0.111; geometry visual mesh filename=package://icub_with_hands/meshes/ll4.dae
- link ll5: mass None -> 0.111; geometry visual mesh filename=package://icub_with_hands/meshes/ll5.dae
- link ll6: mass None -> 0.111; geometry visual mesh filename=package://icub_with_hands/meshes/ll6.dae
- link llil0: mass None -> 0.111; geometry visual mesh filename=package://icub_with_hands/meshes/llil0.dae
- link llil1: mass None -> 0.111; geometry visual mesh filename=package://icub_with_hands/meshes/llil1.dae
- link llil2: mass None -> 0.111; geometry visual mesh filename=package://icub_with_hands/meshes/llil2.dae
- link llil3: mass None -> 0.111; geometry visual mesh filename=package://icub_with_hands/meshes/llil3.dae
- link llittlebase: mass None -> 0.111; geometry visual mesh filename=package://icub_with_hands/meshes/llittlebase.dae
- link lmiddlebase: mass None -> 0.111; geometry visual mesh filename=package://icub_with_hands/meshes/lmiddlebase.dae
- link lml0: mass None -> 0.111; geometry visual mesh filename=package://icub_with_hands/meshes/lml0.dae
- link lml1: mass None -> 0.111; geometry visual mesh filename=package://icub_with_hands/meshes/lml1.dae
- link lml2: mass None -> 0.111; geometry visual mesh filename=package://icub_with_hands/meshes/lml2.dae
- link lml3: mass None -> 0.111; geometry visual mesh filename=package://icub_with_hands/meshes/lml3.dae
- link lril0: mass None -> 0.111; geometry visual mesh filename=package://icub_with_hands/meshes/lril0.dae
- link lril1: mass None -> 0.111; geometry visual mesh filename=package://icub_with_hands/meshes/lril1.dae
- link lril2: mass None -> 0.111; geometry visual mesh filename=package://icub_with_hands/meshes/lril2.dae
- link lril3: mass None -> 0.111; geometry visual mesh filename=package://icub_with_hands/meshes/lril3.dae
- link lringbase: mass None -> 0.111; geometry visual mesh filename=package://icub_with_hands/meshes/lringbase.dae
- link lthumbbase: mass None -> 0.111
- link ltl0: mass None -> 0.111; geometry visual mesh filename=package://icub_with_hands/meshes/ltl0.dae
- link ltl1: mass None -> 0.111; geometry visual mesh filename=package://icub_with_hands/meshes/ltl1.dae
- link ltl2: mass None -> 0.111; geometry visual mesh filename=package://icub_with_hands/meshes/ltl2.dae
- link ltl3: mass None -> 0.111; geometry visual mesh filename=package://icub_with_hands/meshes/ltl3.dae
- link ltl4: mass None -> 0.111; geometry visual mesh filename=package://icub_with_hands/meshes/ltl4.dae
- link middlebase: mass None -> 0.111; geometry visual mesh filename=package://icub_with_hands/meshes/middlebase.dae
- link ml0: mass None -> 0.111; geometry visual mesh filename=package://icub_with_hands/meshes/ml0.dae
- link ml1: mass None -> 0.111; geometry visual mesh filename=package://icub_with_hands/meshes/ml1.dae
- link ml2: mass None -> 0.111; geometry visual mesh filename=package://icub_with_hands/meshes/ml2.dae
- link ml3: mass None -> 0.111; geometry visual mesh filename=package://icub_with_hands/meshes/ml3.dae
- link ra0: mass None -> 0.111; geometry visual mesh filename=package://icub_with_hands/meshes/ra0.dae
- link ra1: mass None -> 0.111; geometry visual mesh filename=package://icub_with_hands/meshes/ra1.dae
- link ra2: mass None -> 0.111; geometry visual mesh filename=package://icub_with_hands/meshes/ra2.dae
- link ra3: mass None -> 0.111; geometry visual mesh filename=package://icub_with_hands/meshes/ra3.dae
- link ra4: mass None -> 0.111; geometry visual mesh filename=package://icub_with_hands/meshes/ra4.dae
- link ra5: mass None -> 0.111; geometry visual mesh filename=package://icub_with_hands/meshes/ra5.dae
- link ra6: mass None -> 0.111; geometry visual mesh filename=package://icub_with_hands/meshes/ra6.dae
- link right_palm: mass None -> 0.111; geometry visual mesh filename=package://icub_with_hands/meshes/right_palm.dae
- link ril0: mass None -> 0.111; geometry visual mesh filename=package://icub_with_hands/meshes/ril0.dae
- link ril1: mass None -> 0.111; geometry visual mesh filename=package://icub_with_hands/meshes/ril1.dae
- link ril2: mass None -> 0.111; geometry visual mesh filename=package://icub_with_hands/meshes/ril2.dae
- link ril3: mass None -> 0.111; geometry visual mesh filename=package://icub_with_hands/meshes/ril3.dae
- link ringbase: mass None -> 0.111; geometry visual mesh filename=package://icub_with_hands/meshes/ringbase.dae
- link rl0: mass None -> 0.111; geometry visual mesh filename=package://icub_with_hands/meshes/rl0.dae
- link rl1: mass None -> 0.111; geometry visual mesh filename=package://icub_with_hands/meshes/rl1.dae
- link rl2: mass None -> 0.111; geometry visual mesh filename=package://icub_with_hands/meshes/rl2.dae
- link rl3: mass None -> 0.111; geometry visual mesh filename=package://icub_with_hands/meshes/rl3.dae
- link rl4: mass None -> 0.111; geometry visual mesh filename=package://icub_with_hands/meshes/rl4.dae
- link rl5: mass None -> 0.111; geometry visual mesh filename=package://icub_with_hands/meshes/rl5.dae
- link rl6: mass None -> 0.111; geometry visual mesh filename=package://icub_with_hands/meshes/rl6.dae
- link thumbbase: mass None -> 0.111
- link tl0: mass None -> 0.111; geometry visual mesh filename=package://icub_with_hands/meshes/tl0.dae
- link tl1: mass None -> 0.111; geometry visual mesh filename=package://icub_with_hands/meshes/tl1.dae
- link tl2: mass None -> 0.111; geometry visual mesh filename=package://icub_with_hands/meshes/tl2.dae
- link tl3: mass None -> 0.111; geometry visual mesh filename=package://icub_with_hands/meshes/tl3.dae
- link tl4: mass None -> 0.111; geometry visual mesh filename=package://icub_with_hands/meshes/tl4.dae
