Commit message: Added option to explicitly assign link masses, and updated model
See https://github.com/robotology/simmechanics-to-urdf/commit/06cdd522c720bd2638bb47acbccf78b3e45d3b6b

File: iCubGenova02/iCubGenova02.urdf (robot description, URDF)
Before this commit: robot iCubGenova02, 99 links, 98 joints
Links:
- link chest: mass 8.63802 -> 7.638
- link l_ankle_1: mass 0.879758 -> 0.6798
- link l_lower_leg: mass 1.87237 -> 1.4724
- link l_upper_leg: mass 2.20843 -> 1.8084
- link r_ankle_1: mass 0.880328 -> 0.6803
- link r_lower_leg: mass 1.87201 -> 1.472
- link r_upper_leg: mass 2.20355 -> 1.8035
Joints:
- joint chest_ems_acc_eb1_fixed_joint: origin xyz=0.0647855001907 0.064043 -0.064709 rpy=3.1415169122972952 -0.2617993091222473 0.0002926418802545251 -> xyz=0.0647855001907 0.064043 -0.064709 rpy=3.1415169123 -0.261799309122 0.000292641880255
- joint chest_ems_acc_eb2_fixed_joint: origin xyz=0.0204533001907 0.088063 -0.0641645 rpy=3.141590501042822 0.2617993198185103 3.1415843367812997 -> xyz=0.0204533001907 0.088063 -0.0641645 rpy=3.14159050104 0.261799319819 3.14158433678
- joint chest_ems_acc_eb3_fixed_joint: origin xyz=-0.0230587998093 0.064019 -0.0758985 rpy=3.141109162025268 0.26110051647116095 -0.00030907146255546275 -> xyz=-0.0230587998093 0.064019 -0.0758985 rpy=3.14110916203 0.261100516471 -0.000309071462555
- joint chest_ems_acc_eb4_fixed_joint: origin xyz=-0.0621620998093 0.088063 -0.0529886 rpy=-3.1415905047625503 -0.26179931981852844 3.141584339870295 -> xyz=-0.0621620998093 0.088063 -0.0529886 rpy=-3.14159050476 -0.261799319819 3.14158433987
- joint chest_ems_gyro_eb1_fixed_joint: origin xyz=0.0692016001907 0.064548 -0.0635257 rpy=3.1415169122972952 -0.2617993091222473 0.0002926418802545251 -> xyz=0.0692016001907 0.064548 -0.0635257 rpy=3.1415169123 -0.261799309122 0.000292641880255
- joint chest_ems_gyro_eb2_fixed_joint: origin xyz=0.0160371001907 0.087559 -0.0653478 rpy=3.141590501042822 0.2617993198185103 3.1415843367812997 -> xyz=0.0160371001907 0.087559 -0.0653478 rpy=3.14159050104 0.261799319819 3.14158433678
- joint chest_ems_gyro_eb3_fixed_joint: origin xyz=-0.0186416998093 0.064521 -0.0770785 rpy=3.141109162025268 0.26110051647116095 -0.00030907146255546275 -> xyz=-0.0186416998093 0.064521 -0.0770785 rpy=3.14110916203 0.261100516471 -0.000309071462555
- joint chest_ems_gyro_eb4_fixed_joint: origin xyz=-0.0665783998093 0.087559 -0.0518053 rpy=-3.1415905047625503 -0.26179931981852844 3.141584339870295 -> xyz=-0.0665783998093 0.087559 -0.0518053 rpy=-3.14159050476 -0.261799319819 3.14158433987
- joint chest_mtb_acc_0b10_fixed_joint: origin xyz=0.0594286001907 -0.0018543 0.0457982 rpy=-0.8751681534754425 0.11636202547856277 -1.6556180750511098 -> xyz=0.0594286001907 -0.0018543 0.0457982 rpy=-0.875168153475 0.116362025479 -1.65561807505
- joint chest_mtb_acc_0b7_fixed_joint: origin xyz=-0.0607539998093 -0.0017836 0.0442342 rpy=0.8751677714915176 0.11636373439232421 -1.485973502467595 -> xyz=-0.0607539998093 -0.0017836 0.0442342 rpy=0.875167771492 0.116363734392 -1.48597350247
- joint chest_mtb_acc_0b8_fixed_joint: origin xyz=-0.0457046998093 -0.001846 0.0567427 rpy=0.5009600846888737 0.10731368898312443 -1.4778325291042227 -> xyz=-0.0457046998093 -0.001846 0.0567427 rpy=0.500960084689 0.107313688983 -1.4778325291
- joint chest_mtb_acc_0b9_fixed_joint: origin xyz=0.0439036001907 -0.0017841 0.0577221 rpy=-0.5009599289728344 0.10731540424780756 -1.663760174692588 -> xyz=0.0439036001907 -0.0017841 0.0577221 rpy=-0.500959928973 0.107315404248 -1.66376017469
- joint imu_frame_fixed_joint: origin xyz=0.00950000019074 0.133444 0.0093 rpy=-1.5707963267948961 1.570796326794896 0 -> xyz=0.00950000019074 0.133444 0.0093 rpy=-1.57079632679 1.57079632679 0
- joint l_ankle_pitch: limit lower=-0.3490658503988659 upper=0.5235987755982988 effort=50000 velocity=50000 -> lower=-0.349065850399 upper=0.523598775598 effort=50000 velocity=50000
- joint l_ankle_roll: limit lower=-0.3490658503988659 upper=0.3490658503988659 effort=50000 velocity=50000 -> lower=-0.349065850399 upper=0.349065850399 effort=50000 velocity=50000
- joint l_arm_ft_sensor: origin xyz=0.0511098470381 2.52343498361e-07 0.0292238157865 rpy=4.5319568084916467e-07 -1.3089970275210927 3.1415921907414344 -> xyz=0.0511098470381 2.52343498361e-07 0.0292238157865 rpy=4.5319568085e-07 -1.30899702752 3.14159219074
- joint l_elbow: limit lower=0.2617993877991494 upper=1.8500490071139892 effort=50000 velocity=50000 -> lower=0.261799387799 upper=1.85004900711 effort=50000 velocity=50000; origin xyz=0 0.0340002020424 0.07926 rpy=0 -1.30899702752112 -3.141592556630374 -> xyz=0 0.0340002020424 0.07926 rpy=0 -1.30899702752 -3.14159255663
- joint l_foot_ft_sensor: origin xyz=0 -0.0603 -0.05158755 rpy=1.5707963267948961 -1.570796326794896 0 -> xyz=0 -0.0603 -0.05158755 rpy=1.57079632679 -1.57079632679 0
- joint l_forearm_mtb_acc_1b7_fixed_joint: origin xyz=0.114369310123 0.0285176341319 -0.016529983678 rpy=0.2617994794375143 0.0003704457632296642 -1.570334469770784 -> xyz=0.114369310123 0.0285176341319 -0.016529983678 rpy=0.261799479438 0.00037044576323 -1.57033446977
- joint l_forearm_mtb_acc_1b8_fixed_joint: origin xyz=0.088920682324 0.0159719572896 0.0352687234784 rpy=-0.6611434090480407 0.14782568634942247 -3.0495222301717226 -> xyz=0.088920682324 0.0159719572896 0.0352687234784 rpy=-0.661143409048 0.147825686349 -3.04952223017
- joint l_forearm_mtb_acc_1b9_fixed_joint: origin xyz=0.0595956869538 0.0596564434985 -0.0205993985252 rpy=1.7668208948349358 0.2611001649697097 3.0875256913488913 -> xyz=0.0595956869538 0.0596564434985 -0.0205993985252 rpy=1.76682089483 0.26110016497 3.08752569135
- joint l_hip_pitch: limit lower=-0.5235987755982988 upper=1.4835298641951802 effort=50000 velocity=50000 -> lower=-0.523598775598 upper=1.4835298642 effort=50000 velocity=50000; origin xyz=0.0064515 -0.0223861 -0.119913 rpy=1.5707963267948961 0 -1.5707963267948961 -> xyz=0.0064515 -0.0223861 -0.119913 rpy=1.57079632679 0 -1.57079632679
- joint l_hip_roll: limit lower=0.0 upper=1.5707963267948966 effort=50000 velocity=50000 -> lower=0.0 upper=1.57079632679 effort=50000 velocity=50000
- joint l_hip_yaw: limit lower=-1.2217304763960306 upper=1.2217304763960306 effort=50000 velocity=50000 -> lower=-1.2217304764 upper=1.2217304764 effort=50000 velocity=50000; origin xyz=0 0 0.0146 rpy=-1.5707963267948961 0 -1.5707963267948961 -> xyz=0 0 0.0146 rpy=-1.57079632679 0 -1.57079632679
- joint l_knee: axis -1.0 0.0 0.0 -> -1.0 -0.0 -0.0; limit lower=-1.7453292519943295 upper=0.0 effort=50000 velocity=50000 -> lower=-1.74532925199 upper=0.0 effort=50000 velocity=50000
- joint l_leg_ft_sensor: origin xyz=0 -0.0743 0.0246825 rpy=1.5707963267948961 -1.570796326794896 0 -> xyz=0 -0.0743 0.0246825 rpy=1.57079632679 -1.57079632679 0
- joint l_lower_leg_ems_acc_eb7_fixed_joint: origin xyz=0.0350978 -0.092765 0.04351373 rpy=0 -0.21816654334094113 1.5707963267948974 -> xyz=0.0350978 -0.092765 0.04351373 rpy=0 -0.218166543341 1.57079632679
- joint l_lower_leg_ems_gyro_eb7_fixed_joint: origin xyz=0.0356017 -0.088301 0.044503292 rpy=0 -0.21816654334094113 1.5707963267948974 -> xyz=0.0356017 -0.088301 0.044503292 rpy=0 -0.218166543341 1.57079632679
- joint l_lower_leg_mtb_acc_10b10_fixed_joint: origin xyz=0.030989 -0.011037 0.05238133 rpy=-1.326450423673184 0 1.5707963267948961 -> xyz=0.030989 -0.011037 0.05238133 rpy=-1.32645042367 0 1.57079632679
- joint l_lower_leg_mtb_acc_10b11_fixed_joint: origin xyz=-0.0179355 -0.092958 0.0184593 rpy=-1.3089971472018722 -2.543178857158298e-05 1.5707895123459004 -> xyz=-0.0179355 -0.092958 0.0184593 rpy=-1.3089971472 -2.54317885716e-05 1.57078951235
- joint l_lower_leg_mtb_acc_10b8_fixed_joint: origin xyz=0.0099841 -0.004318 0.0544518 rpy=-0.34906563804548707 3.9714103784092166e-05 1.570905440483374 -> xyz=0.0099841 -0.004318 0.0544518 rpy=-0.349065638045 3.97141037841e-05 1.57090544048
- joint l_lower_leg_mtb_acc_10b9_fixed_joint: origin xyz=0.0665272 -0.043468 0.0259151 rpy=1.30899714593518 -0.00011215980287766697 1.5708263802148703 -> xyz=0.0665272 -0.043468 0.0259151 rpy=1.30899714594 -0.000112159802878 1.57082638021
- joint l_shoulder_pitch: limit lower=-1.6667894356545847 upper=0.17453292519943295 effort=50000 velocity=50000 -> lower=-1.66678943565 upper=0.174532925199 effort=50000 velocity=50000
- joint l_shoulder_roll: limit lower=0.0 upper=2.8064894372068823 effort=50000 velocity=50000 -> lower=0.0 upper=2.80648943721 effort=50000 velocity=50000; origin xyz=-0.013671 0 0.0085203 rpy=0.2705973179159596 0.25268017754236044 -1.5015568855866173 -> xyz=-0.013671 0 0.0085203 rpy=0.270597317916 0.252680177542 -1.50155688559
- joint l_shoulder_yaw: limit lower=-0.6457718232379019 upper=1.3962634015954636 effort=50000 velocity=50000 -> lower=-0.645771823238 upper=1.3962634016 effort=50000 velocity=50000
- joint l_upper_arm_mtb_acc_1b10_fixed_joint: origin xyz=-0.0430553865107 -0.0286807251034 0.0295279 rpy=-1.570796460941082 -1.5705035075902931 2.6825718625443584 -> xyz=-0.0430553865107 -0.0286807251034 0.0295279 rpy=-1.57079646094 -1.57050350759 2.68257186254
- joint l_upper_arm_mtb_acc_1b11_fixed_joint: origin xyz=-0.0412179516256 -0.0295882096119 0.0760604 rpy=-1.570796460941082 -1.5705035075902931 2.6825718625443584 -> xyz=-0.0412179516256 -0.0295882096119 0.0760604 rpy=-1.57079646094 -1.57050350759 2.68257186254
- joint l_upper_arm_mtb_acc_1b12_fixed_joint: origin xyz=-0.0412194005144 -0.0295878213836 0.0049921 rpy=-1.5707956830363743 -1.570783812267946 2.682571084586891 -> xyz=-0.0412194005144 -0.0295878213836 0.0049921 rpy=-1.57079568304 -1.57078381227 2.68257108459
- joint l_upper_arm_mtb_acc_1b13_fixed_joint: origin xyz=0.0105927619825 -0.0283506291435 -0.0086914 rpy=-1.5707963266769467 0.00021452011106801812 -2.4780369107521003 -> xyz=0.0105927619825 -0.0283506291435 -0.0086914 rpy=-1.57079632668 0.000214520111068 -2.47803691075
- joint l_upper_leg_ems_acc_eb10_fixed_joint: origin xyz=0.040407 -0.040027 -0.0125751 rpy=1.5707963267948961 0 1.5707963267948961 -> xyz=0.040407 -0.040027 -0.0125751 rpy=1.57079632679 0 1.57079632679
- joint l_upper_leg_ems_acc_eb6_fixed_joint: origin xyz=-0.0404072 -0.083207 -0.0125771 rpy=1.5707963267948961 0 -1.5707963267948961 -> xyz=-0.0404072 -0.083207 -0.0125771 rpy=1.57079632679 0 -1.57079632679
- joint l_upper_leg_ems_gyro_eb10_fixed_joint: origin xyz=0.040407 -0.035455 -0.013079 rpy=1.5707963267948961 0 1.5707963267948961 -> xyz=0.040407 -0.035455 -0.013079 rpy=1.57079632679 0 1.57079632679
- joint l_upper_leg_ems_gyro_eb6_fixed_joint: origin xyz=-0.0404072 -0.087779 -0.013081 rpy=1.5707963267948961 0 -1.5707963267948961 -> xyz=-0.0404072 -0.087779 -0.013081 rpy=1.57079632679 0 -1.57079632679
- joint l_upper_leg_mtb_acc_10b1_fixed_joint: origin xyz=0.031565 0.049332 0.04200163 rpy=0.8377580369611062 -8.629128296517655e-05 1.5708740239417236 -> xyz=0.031565 0.049332 0.04200163 rpy=0.837758036961 -8.62912829653e-05 1.57087402394
- joint l_upper_leg_mtb_acc_10b2_fixed_joint: origin xyz=0.0083839 0.039452 0.05335544 rpy=0.8377580369650546 -8.629128691368476e-05 1.5708740239399657 -> xyz=0.0083839 0.039452 0.05335544 rpy=0.837758036965 -8.62912869137e-05 1.57087402394
- joint l_upper_leg_mtb_acc_10b3_fixed_joint: origin xyz=0.0150706 0.004382 0.053785 rpy=0 0 1.5707963267948966 -> xyz=0.0150706 0.004382 0.053785 rpy=0 0 1.57079632679
- joint l_upper_leg_mtb_acc_10b4_fixed_joint: origin xyz=-0.0144294 0.004382 0.053785 rpy=0 0 1.5707963267948966 -> xyz=-0.0144294 0.004382 0.053785 rpy=0 0 1.57079632679
- joint l_upper_leg_mtb_acc_10b5_fixed_joint: origin xyz=-0.0414999 -0.004658 0.03412949 rpy=-1.186823762544959 0 1.5707963267948963 -> xyz=-0.0414999 -0.004658 0.03412949 rpy=-1.18682376254 0 1.57079632679
- joint l_upper_leg_mtb_acc_10b6_fixed_joint: origin xyz=0.0178086 -0.026212 -0.043785 rpy=3.141592653589793 0 -1.5709124300543913 -> xyz=0.0178086 -0.026212 -0.043785 rpy=3.14159265359 0 -1.57091243005
- joint l_upper_leg_mtb_acc_10b7_fixed_joint: origin xyz=-0.0141918 -0.026211 -0.043785 rpy=3.141592653589793 0 -1.5709453146950971 -> xyz=-0.0141918 -0.026211 -0.043785 rpy=3.14159265359 0 -1.5709453147
- joint neck_pitch: limit lower=-0.6981317007977318 upper=0.3839724354387525 effort=50000 velocity=50000 -> lower=-0.698131700798 upper=0.383972435439 effort=50000 velocity=50000
- joint neck_roll: limit lower=-0.3490658503988659 upper=0.3490658503988659 effort=50000 velocity=50000 -> lower=-0.349065850399 upper=0.349065850399 effort=50000 velocity=50000
- joint neck_yaw: limit lower=-0.8726646259971648 upper=0.8726646259971648 effort=50000 velocity=50000 -> lower=-0.872664625997 upper=0.872664625997 effort=50000 velocity=50000
- joint r_ankle_pitch: limit lower=-0.3490658503988659 upper=0.5235987755982988 effort=50000 velocity=50000 -> lower=-0.349065850399 upper=0.523598775598 effort=50000 velocity=50000
- joint r_ankle_roll: axis 0.0 0.0 -1.0 -> -0.0 -0.0 -1.0; limit lower=-0.3490658503988659 upper=0.3490658503988659 effort=50000 velocity=50000 -> lower=-0.349065850399 upper=0.349065850399 effort=50000 velocity=50000
- joint r_arm_ft_sensor: origin xyz=-0.0513445670194 2.52344985144e-07 0.0292867087936 rpy=-4.5319568070266037e-07 -1.3089970275210934 4.628483589970802e-07 -> xyz=-0.0513445670194 2.52344985144e-07 0.0292867087936 rpy=-4.5319568147e-07 -1.30899702752 4.62848360172e-07
- joint r_elbow: limit lower=0.2617993877991494 upper=1.8500490071139892 effort=50000 velocity=50000 -> lower=0.261799387799 upper=1.85004900711 effort=50000 velocity=50000; origin xyz=0 -0.0225001557729 0.07926 rpy=0 1.308997027521121 0 -> xyz=0 -0.0225001557729 0.07926 rpy=0 1.30899702752 0
- joint r_foot_ft_sensor: origin xyz=0 -0.0603 0.015 rpy=1.5707963267948961 -1.570796326794896 0 -> xyz=0 -0.0603 0.015 rpy=1.57079632679 -1.57079632679 0
- joint r_foot_mtb_acc_11b12_fixed_joint: origin xyz=0.1034744 -0.000807 -0.001215 rpy=0 0 -1.5707963267948966 -> xyz=0.1034744 -0.000807 -0.001215 rpy=0 0 -1.57079632679
- joint r_foot_mtb_acc_11b13_fixed_joint: origin xyz=0.0784744 -0.0118072 -0.001215 rpy=0 0 -1.5707963267948966 -> xyz=0.0784744 -0.0118072 -0.001215 rpy=0 0 -1.57079632679
- joint r_forearm_mtb_acc_2b7_fixed_joint: origin xyz=-0.11436927713 0.0279967173307 -0.0165298605327 rpy=0.2617994793812094 0.00037025313277796464 1.5712581194176245 -> xyz=-0.11436927713 0.0279967173307 -0.0165298605327 rpy=0.261799479381 0.000370253132778 1.57125811942
- joint r_forearm_mtb_acc_2b8_fixed_joint: origin xyz=-0.0891879779927 0.00375149154266 0.0348004899258 rpy=0.6611590015134917 0.14774579417419006 -0.0919672808581299 -> xyz=-0.0891879779927 0.00375149154266 0.0348004899258 rpy=0.661159001513 0.147745794174 -0.0919672808581
- joint r_forearm_mtb_acc_2b9_fixed_joint: origin xyz=-0.0591344983628 0.0504236337681 -0.0187310112996 rpy=-1.7668262973366173 0.26119181238162653 0.05404748777229077 -> xyz=-0.0591344983628 0.0504236337681 -0.0187310112996 rpy=-1.76682629734 0.261191812382 0.0540474877723
- joint r_hip_pitch: axis -1.0 0.0 0.0 -> -1.0 -0.0 -0.0; limit lower=-0.5235987755982988 upper=1.4835298641951802 effort=50000 velocity=50000 -> lower=-0.523598775598 upper=1.4835298642 effort=50000 velocity=50000; origin xyz=0.0064515 0.0233655 -0.119913 rpy=1.5707963267948961 0 -1.5707963267948961 -> xyz=0.0064515 0.0233655 -0.119913 rpy=1.57079632679 0 -1.57079632679
- joint r_hip_roll: axis 0.0 0.0 -1.0 -> -0.0 -0.0 -1.0; limit lower=0.0 upper=1.5707963267948966 effort=50000 velocity=50000 -> lower=0.0 upper=1.57079632679 effort=50000 velocity=50000
- joint r_hip_yaw: limit lower=-1.2217304763960306 upper=1.2217304763960306 effort=50000 velocity=50000 -> lower=-1.2217304764 upper=1.2217304764 effort=50000 velocity=50000; origin xyz=0 0 0.0146 rpy=-1.5707963267948961 0 -1.5707963267948961 -> xyz=0 0 0.0146 rpy=-1.57079632679 0 -1.57079632679
- joint r_knee: limit lower=-1.7453292519943295 upper=0.0 effort=50000 velocity=50000 -> lower=-1.74532925199 upper=0.0 effort=50000 velocity=50000
- joint r_leg_ft_sensor: origin xyz=0 -0.0743 0.0254872 rpy=1.5707963267948961 -1.570796326794896 0 -> xyz=0 -0.0743 0.0254872 rpy=1.57079632679 -1.57079632679 0
- joint r_lower_leg_ems_acc_eb9_fixed_joint: origin xyz=-0.0099643 -0.092765 0.04351373 rpy=0 -0.21816654334094113 1.5707963267948974 -> xyz=-0.0099643 -0.092765 0.04351373 rpy=0 -0.218166543341 1.57079632679
- joint r_lower_leg_ems_gyro_eb9_fixed_joint: origin xyz=-0.0094604 -0.088301 0.044503292 rpy=0 -0.21816654334094113 1.5707963267948974 -> xyz=-0.0094604 -0.088301 0.044503292 rpy=0 -0.218166543341 1.57079632679
- joint r_lower_leg_mtb_acc_11b10_fixed_joint: origin xyz=-0.0389997 -0.004318 0.05362922 rpy=-0.2443461645654741 2.8091104096089837e-05 1.5709089943462522 -> xyz=-0.0389997 -0.004318 0.05362922 rpy=-0.244346164565 2.80911040962e-05 1.57090899435
- joint r_lower_leg_mtb_acc_11b11_fixed_joint: origin xyz=0.0184451 -0.092958 0.0164801 rpy=1.30899714593518 -0.00011215980287766697 1.5708263802148703 -> xyz=0.0184451 -0.092958 0.0164801 rpy=1.30899714594 -0.000112159802878 1.57082638021
- joint r_lower_leg_mtb_acc_11b8_fixed_joint: origin xyz=-0.008081 -0.004318 0.0537517 rpy=0.34906563804609786 -3.971410439477034e-05 1.5709054404832665 -> xyz=-0.008081 -0.004318 0.0537517 rpy=0.349065638046 -3.97141043948e-05 1.57090544048
- joint r_lower_leg_mtb_acc_11b9_fixed_joint: origin xyz=-0.0660179 -0.043468 0.0278945 rpy=-1.3089971473150512 0 1.5707963267948968 -> xyz=-0.0660179 -0.043468 0.0278945 rpy=-1.30899714732 0 1.57079632679
- joint r_shoulder_pitch: limit lower=-1.6667894356545847 upper=0.17453292519943295 effort=50000 velocity=50000 -> lower=-1.66678943565 upper=0.174532925199 effort=50000 velocity=50000; origin xyz=-0.120015999809 0.0928 0.0079694 rpy=0 -0.523598883792035 3.141592653589793 -> xyz=-0.120015999809 0.0928 0.0079694 rpy=0 -0.523598883792 3.14159265359
- joint r_shoulder_roll: limit lower=0.0 upper=2.8064894372068823 effort=50000 velocity=50000 -> lower=0.0 upper=2.80648943721 effort=50000 velocity=50000; origin xyz=-0.00758046573227 0 0.0142102463639 rpy=-0.2705976115829963 -0.252680154648383 -1.5015568003498745 -> xyz=-0.00758046573227 0 0.0142102463639 rpy=-0.270597611583 -0.252680154648 -1.50155680035
- joint r_shoulder_yaw: limit lower=-0.6457718232379019 upper=1.3962634015954636 effort=50000 velocity=50000 -> lower=-0.645771823238 upper=1.3962634016 effort=50000 velocity=50000
- joint r_sole_fixed_joint: origin xyz=0.0035 0 0.004 rpy=-3.141592653589793 0 0 -> xyz=0.0035 0 0.004 rpy=-3.14159265359 0 0
- joint r_upper_arm_mtb_acc_2b10_fixed_joint: origin xyz=-0.0412194005144 0.0295878213836 0.0295279 rpy=1.5707969705667262 1.5707838122679458 -2.682571084564997 -> xyz=-0.0412194005144 0.0295878213836 0.0295279 rpy=1.5707969706 1.57078381227 -2.68257108456
- joint r_upper_arm_mtb_acc_2b11_fixed_joint: origin xyz=-0.0430565765807 0.0286793709492 0.0760604 rpy=-1.5707961926490903 -1.5705035075902927 0.4590207910451026 -> xyz=-0.0430565765807 0.0286793709492 0.0760604 rpy=-1.57079619265 -1.57050350759 0.459020791048
- joint r_upper_arm_mtb_acc_2b12_fixed_joint: origin xyz=-0.0430553865107 0.0286807251034 0.0049922 rpy=-1.111775401564534 -1.5707963267948961 0 -> xyz=-0.0430553865107 0.0286807251034 0.0049922 rpy=-1.98902065637 -1.57079632679 0.785398163397
- joint r_upper_arm_mtb_acc_2b13_fixed_joint: origin xyz=0.010593416831 0.0283497693333 -0.010738 rpy=1.5707963269128467 -0.00021452011106801806 2.4780369107521003 -> xyz=0.010593416831 0.0283497693333 -0.010738 rpy=1.57079632691 -0.000214520111068 2.47803691075
- joint r_upper_leg_ems_acc_eb11_fixed_joint: origin xyz=-0.040407 -0.083207 -0.0125771 rpy=1.5707963267948961 0 -1.5707963267948961 -> xyz=-0.040407 -0.083207 -0.0125771 rpy=1.57079632679 0 -1.57079632679
- joint r_upper_leg_ems_acc_eb8_fixed_joint: origin xyz=0.0404072 -0.040027 -0.0125751 rpy=1.5707963267948961 0 -1.5707963267948961 -> xyz=0.0404072 -0.040027 -0.0125751 rpy=1.57079632679 0 -1.57079632679
- joint r_upper_leg_ems_gyro_eb11_fixed_joint: origin xyz=-0.040407 -0.087779 -0.013081 rpy=1.5707963267948961 0 -1.5707963267948961 -> xyz=-0.040407 -0.087779 -0.013081 rpy=1.57079632679 0 -1.57079632679
- joint r_upper_leg_ems_gyro_eb8_fixed_joint: origin xyz=0.0404072 -0.035455 -0.013079 rpy=1.5707963267948961 0 -1.5707963267948961 -> xyz=0.0404072 -0.035455 -0.013079 rpy=1.57079632679 0 -1.57079632679
- joint r_upper_leg_mtb_acc_11b1_fixed_joint: origin xyz=-0.030195 0.04914 0.043588612 rpy=-0.8377580538579834 -0.0003427907493437384 1.570874016517316 -> xyz=-0.030195 0.04914 0.043588612 rpy=-0.837758053858 -0.000342790749344 1.57087401652
- joint r_upper_leg_mtb_acc_11b2_fixed_joint: origin xyz=-0.0064065 0.039256 0.0539467 rpy=-0.8377580538579834 -0.0003427907493437384 1.570874016517316 -> xyz=-0.0064065 0.039256 0.0539467 rpy=-0.837758053858 -0.000342790749344 1.57087401652
- joint r_upper_leg_mtb_acc_11b3_fixed_joint: origin xyz=-0.0130214 0.004186 0.0538313 rpy=0 -0.00042908999059361946 1.570912443546613 -> xyz=-0.0130214 0.004186 0.0538313 rpy=0 -0.000429089990594 1.57091244355
- joint r_upper_leg_mtb_acc_11b4_fixed_joint: origin xyz=0.0422675 -0.004845 0.0322719 rpy=1.1868237508623853 -0.0005368537261927895 1.5708398310564209 -> xyz=0.0422675 -0.004845 0.0322719 rpy=1.18682375086 -0.000536853726193 1.57083983106
- joint r_upper_leg_mtb_acc_11b5_fixed_joint: origin xyz=0.0164786 0.004186 0.0538313 rpy=0 -0.00042908999059361946 1.570912443546613 -> xyz=0.0164786 0.004186 0.0538313 rpy=0 -0.000429089990594 1.57091244355
- joint r_upper_leg_mtb_acc_11b6_fixed_joint: origin xyz=-0.0157594 -0.026365 -0.0437518 rpy=3.141592653589793 0.0004290899934163925 -1.5707963267948968 -> xyz=-0.0157594 -0.026365 -0.0437518 rpy=3.14159265359 0.000429089993416 -1.57079632679
- joint r_upper_leg_mtb_acc_11b7_fixed_joint: origin xyz=0.0162386 -0.026366 -0.0437518 rpy=3.1415926037711634 0.000429089990404397 -1.5709124300650796 -> xyz=0.0162386 -0.026366 -0.0437518 rpy=3.14159260377 0.000429089990404 -1.57091243007
- joint root_link_ems_acc_eb5_fixed_joint: origin xyz=0.0493308 -0.0125771 -0.115691 rpy=3.141592653589793 1.2915440450258349 3.141592653589793 -> xyz=0.0493308 -0.0125771 -0.115691 rpy=3.14159265359 1.29154404503 3.14159265359
- joint root_link_ems_gyro_eb5_fixed_joint: origin xyz=0.0493308 -0.0125771 -0.115691 rpy=3.141592653589793 1.2915440450258349 3.141592653589793 -> xyz=0.0493308 -0.0125771 -0.115691 rpy=3.14159265359 1.29154404503 3.14159265359
- joint torso_pitch: limit lower=-0.3490658503988659 upper=1.2217304763960306 effort=50000 velocity=50000 -> lower=-0.349065850399 upper=1.2217304764 effort=50000 velocity=50000; origin xyz=0 0.0270463 0 rpy=1.5707963267948961 0 -1.5707963267948961 -> xyz=0 0.0270463 0 rpy=1.57079632679 0 -1.57079632679
- joint torso_roll: limit lower=-0.5235987755982988 upper=0.5235987755982988 effort=50000 velocity=50000 -> lower=-0.523598775598 upper=0.523598775598 effort=50000 velocity=50000
- joint torso_yaw: limit lower=-0.8726646259971648 upper=0.8726646259971648 effort=50000 velocity=50000 -> lower=-0.872664625997 upper=0.872664625997 effort=50000 velocity=50000
