Commit message: adding missing frames in left foot changed zero position for shoulder yaw - to be checked

File: iCubGenova02/iCubGenova02.urdf (robot description, URDF)
Before this commit: robot iCubGenova02, 99 links, 98 joints
Links:
- added link l_foot_mtb_acc_10b12
- added link l_foot_mtb_acc_10b13
- added link l_sole
Joints:
- added joint l_foot_mtb_acc_10b12_fixed_joint: type fixed, parent l_foot, child l_foot_mtb_acc_10b12, origin xyz=0.1055224 0.0008072 -0.001215 rpy=0 0 1.57079632679
- added joint l_foot_mtb_acc_10b13_fixed_joint: type fixed, parent l_foot, child l_foot_mtb_acc_10b13, origin xyz=0.0805224 0.0118072 -0.001215 rpy=0 0 1.57079632679
- added joint l_sole_fixed_joint: type fixed, parent l_foot, child l_sole, origin xyz=0.0035 0 0.004 rpy=-3.14159265359 0 0
- joint l_arm_ft_sensor: origin xyz=0.0511098470381 2.52343498361e-07 0.0292238157865 rpy=4.5319568085e-07 -1.30899702752 3.14159219074 -> xyz=0.0516613635958 0 0.0293716941036 rpy=-1.74628392948e-06 -1.30899688162 -3.14159105254
- joint l_elbow: axis 5.91000555439e-09 -1.00000015612 1.58358068325e-09 -> -1.37984003487e-07 -0.999999650312 -2.56958662737e-07; origin xyz=0 0.0340002020424 0.07926 rpy=0 -1.30899702752 -3.14159255663 -> xyz=0 0.0339999448094 0.07926 rpy=-7.71922125831e-07 -1.30899688162 -3.14159232235
- joint l_forearm_mtb_acc_1b7_fixed_joint: origin xyz=0.114369310123 0.0285176341319 -0.016529983678 rpy=0.261799479438 0.00037044576323 -1.57033446977 -> xyz=0.114369345693 0.0285175082586 -0.0165300680535 rpy=0.261799625374 0.00037007465458 -1.57033478257
- joint l_forearm_mtb_acc_1b8_fixed_joint: origin xyz=0.088920682324 0.0159719572896 0.0352687234784 rpy=-0.661143409048 0.147825686349 -3.04952223017 -> xyz=0.0889206610948 0.0159719646979 0.0352688091831 rpy=-0.661143706905 0.147825404276 -3.04952288278
- joint l_forearm_mtb_acc_1b9_fixed_joint: origin xyz=0.0595956869538 0.0596564434985 -0.0205993985252 rpy=1.76682089483 0.26110016497 3.08752569135 -> xyz=0.0595956740027 0.059656277851 -0.0205992828194 rpy=1.76682145584 0.261100257657 3.08752517336
- joint l_knee: axis -1.0 -0.0 -0.0 -> -1.0 0.0 0.0
- joint l_shoulder_yaw: axis 0.965925849201 6.1184868283e-09 0.258818959594 -> 0.96592581144 -1.99788190436e-07 0.258819100522; origin xyz=0.0251346596233 1.37517196103e-07 -0.00544866358786 rpy=0 0 0 -> xyz=0.0245831159634 1.37513702453e-07 -0.00559644921379 rpy=0.252689649873 -0.00851855576128 0.0670401609012
- joint l_upper_arm_mtb_acc_1b10_fixed_joint: origin xyz=-0.0430553865107 -0.0286807251034 0.0295279 rpy=-1.57079646094 -1.57050350759 2.68257186254 -> xyz=-0.0430554367139 -0.0286807664868 0.0295279 rpy=-1.57079583952 -1.5705035075 2.68256977965
- joint l_upper_arm_mtb_acc_1b11_fixed_joint: origin xyz=-0.0412179516256 -0.0295882096119 0.0760604 rpy=-1.57079646094 -1.57050350759 2.68257186254 -> xyz=-0.0412183285273 -0.0295890018753 0.0760604 rpy=-1.57079583952 -1.5705035075 2.68256977965
- joint l_upper_arm_mtb_acc_1b12_fixed_joint: origin xyz=-0.0412194005144 -0.0295878213836 0.0049921 rpy=-1.57079568304 -1.57078381227 2.68257108459 -> xyz=-0.0412196275651 -0.0295882518747 0.0049921 rpy=-1.5707932288 -1.57078381223 2.68256716904
- joint l_upper_arm_mtb_acc_1b13_fixed_joint: origin xyz=0.0105927619825 -0.0283506291435 -0.0086914 rpy=-1.57079632668 0.000214520111068 -2.47803691075 -> xyz=0.0105927291029 -0.0283506394525 -0.0086914 rpy=-1.57079632675 0.000214519949312 -2.47803722745
- joint r_ankle_roll: axis -0.0 -0.0 -1.0 -> 0.0 0.0 -1.0
- joint r_arm_ft_sensor: origin xyz=-0.0513445670194 2.52344985144e-07 0.0292867087936 rpy=-4.5319568147e-07 -1.30899702752 4.62848360172e-07 -> xyz=-0.0563122963778 0 0.0306179080726 rpy=1.74628392902e-06 -1.30899688162 -1.60105022579e-06
- joint r_elbow: axis 5.91000555439e-09 1.00000015612 -1.58358068325e-09 -> -1.37984003487e-07 0.999999650312 2.56958662737e-07; origin xyz=0 -0.0225001557729 0.07926 rpy=0 1.30899702752 0 -> xyz=0 -0.0224999380055 0.07926 rpy=-7.71922126771e-07 1.30899688162 -3.31237127341e-07
- joint r_forearm_mtb_acc_2b7_fixed_joint: origin xyz=-0.11436927713 0.0279967173307 -0.0165298605327 rpy=0.261799479381 0.000370253132778 1.57125811942 -> xyz=-0.114369265311 0.0279965709939 -0.0165297684653 rpy=0.261799625193 0.000369941711734 1.57125824894
- joint r_forearm_mtb_acc_2b8_fixed_joint: origin xyz=-0.0891879779927 0.00375149154266 0.0348004899258 rpy=0.661159001513 0.147745794174 -0.0919672808581 -> xyz=-0.0891879834272 0.00375155404808 0.0348004666918 rpy=0.661159497398 0.147746404879 -0.0919671561069
- joint r_forearm_mtb_acc_2b9_fixed_joint: origin xyz=-0.0591344983628 0.0504236337681 -0.0187310112996 rpy=-1.76682629734 0.261191812382 0.0540474877723 -> xyz=-0.0591345608219 0.0504239784737 -0.0187311854579 rpy=-1.76682610154 0.261191762274 0.054048079594
- joint r_hip_pitch: axis -1.0 -0.0 -0.0 -> -1.0 0.0 0.0
- joint r_hip_roll: axis -0.0 -0.0 -1.0 -> 0.0 0.0 -1.0
- joint r_shoulder_yaw: axis 0.965925849201 -6.1184868283e-09 -0.258818959594 -> 0.96592581144 1.99788190436e-07 -0.258819100522; origin xyz=-0.024898847655 2.32747594447e-07 -0.00550748124286 rpy=0 0 0 -> xyz=-0.0199310910125 2.32716127063e-07 -0.00683858715205 rpy=0.252689649873 0.00851855576128 -0.0670401609012
- joint r_upper_arm_mtb_acc_2b10_fixed_joint: origin xyz=-0.0412194005144 0.0295878213836 0.0295279 rpy=1.5707969706 1.57078381227 -2.68257108456 -> xyz=-0.0412196275651 0.0295882518747 0.0295279 rpy=1.57079942481 1.57078381208 -2.6825671691
- joint r_upper_arm_mtb_acc_2b11_fixed_joint: origin xyz=-0.0430565765807 0.0286793709492 0.0760604 rpy=-1.57079619265 -1.57050350759 0.459020791048 -> xyz=-0.0430568223542 0.0286799664862 0.0760604 rpy=-1.57079681407 -1.5705035075 0.459022873944
- joint r_upper_arm_mtb_acc_2b12_fixed_joint: origin xyz=-0.0430553865107 0.0286807251034 0.0049922 rpy=-1.98902065637 -1.57079632679 0.785398163397 -> xyz=-0.0430555233164 0.0286807164867 0.0049922 rpy=-1.11177394027 -1.57079632679 0
- joint r_upper_arm_mtb_acc_2b13_fixed_joint: origin xyz=0.010593416831 0.0283497693333 -0.010738 rpy=1.57079632691 -0.000214520111068 2.47803691075 -> xyz=0.0105929889104 0.0283507894526 -0.010738 rpy=1.57079632684 -0.000214519949312 2.47803722745

Commit message: various fixes to the iCubGenova02 model

File: iCubGenova02/iCubGenova02.urdf (robot description, URDF)
Before this commit: robot iCubGenova02, 99 links, 98 joints
Links:
- added link l_foot_mtb_acc_10b12
- added link l_foot_mtb_acc_10b13
- added link l_sole
Joints:
- added joint l_foot_mtb_acc_10b12_fixed_joint: type fixed, parent l_foot, child l_foot_mtb_acc_10b12, origin xyz=0.1055224 0.0008072 -0.001215 rpy=0 0 1.57079632679
- added joint l_foot_mtb_acc_10b13_fixed_joint: type fixed, parent l_foot, child l_foot_mtb_acc_10b13, origin xyz=0.0805224 0.0118072 -0.001215 rpy=0 0 1.57079632679
- added joint l_sole_fixed_joint: type fixed, parent l_foot, child l_sole, origin xyz=0.0035 0 0.004 rpy=-3.14159265359 0 0
- joint l_arm_ft_sensor: origin xyz=0.0511098470381 2.52343498361e-07 0.0292238157865 rpy=4.5319568085e-07 -1.30899702752 3.14159219074 -> xyz=0.0509301432452 0 0.0291758294659 rpy=0 -1.30899700697 3.14159265359
- joint l_elbow: axis 5.91000555439e-09 -1.00000015612 1.58358068325e-09 -> 2.22044604925e-16 -1.0 0.0; origin xyz=0 0.0340002020424 0.07926 rpy=0 -1.30899702752 -3.14159255663 -> xyz=0 0.0339999 0.07926 rpy=0 -1.30899700697 -3.14159265359
- joint l_forearm_mtb_acc_1b7_fixed_joint: origin xyz=0.114369310123 0.0285176341319 -0.016529983678 rpy=0.261799479438 0.00037044576323 -1.57033446977 -> xyz=0.114369314675 0.0285169 -0.0165299963729 rpy=0.26179949998 0.000370413042328 -1.57033448496
- joint l_forearm_mtb_acc_1b8_fixed_joint: origin xyz=0.088920682324 0.0159719572896 0.0352687234784 rpy=-0.661143409048 0.147825686349 -3.04952223017 -> xyz=0.088920691578 0.015972 0.035268688442 rpy=-0.661143946092 0.147825248461 -3.04952253889
- joint l_forearm_mtb_acc_1b9_fixed_joint: origin xyz=0.0595956869538 0.0596564434985 -0.0205993985252 rpy=1.76682089483 0.26110016497 3.08752569135 -> xyz=0.0595957174403 0.0596569 -0.0205995080872 rpy=1.76682134218 0.261099829847 3.08752548202
- joint l_shoulder_yaw: axis 0.965925849201 6.1184868283e-09 0.258818959594 -> 0.965925843882 2.22044604925e-16 0.258818979447; origin xyz=0.0251346596233 1.37517196103e-07 -0.00544866358786 rpy=0 0 0 -> xyz=0.0253143218312 1.37518334151e-07 -0.00540052326137 rpy=-0.252689546175 -0.0085186183214 -0.067039889142
- joint l_upper_arm_mtb_acc_1b10_fixed_joint: origin xyz=-0.0430553865107 -0.0286807251034 0.0295279 rpy=-1.57079646094 -1.57050350759 2.68257186254 -> xyz=-0.0430554 -0.028681 0.0295279 rpy=-1.57079650664 -1.57050350741 2.68257092837
- joint l_upper_arm_mtb_acc_1b11_fixed_joint: origin xyz=-0.0412179516256 -0.0295882096119 0.0760604 rpy=-1.57079646094 -1.57050350759 2.68257186254 -> xyz=-0.0412181 -0.029589 0.0760604 rpy=-1.57079650664 -1.57050350741 2.68257092837
- joint l_upper_arm_mtb_acc_1b12_fixed_joint: origin xyz=-0.0412194005144 -0.0295878213836 0.0049921 rpy=-1.57079568304 -1.57078381227 2.68257108459 -> xyz=-0.0412195 -0.029588 0.0049921 rpy=-1.57079718993 -1.57078381225 2.68257161162
- joint l_upper_arm_mtb_acc_1b13_fixed_joint: origin xyz=0.0105927619825 -0.0283506291435 -0.0086914 rpy=-1.57079632668 0.000214520111068 -2.47803691075 -> xyz=0.010592657 -0.028351 -0.0086914 rpy=-1.57079632657 0.000214520362042 -2.47803674451
- joint r_arm_ft_sensor: origin xyz=-0.0513445670194 2.52344985144e-07 0.0292867087936 rpy=-4.5319568147e-07 -1.30899702752 4.62848360172e-07 -> xyz=-0.0508973017665 0 0.0291670296206 rpy=0 -1.30899700697 0
- joint r_elbow: axis 5.91000555439e-09 1.00000015612 -1.58358068325e-09 -> 2.22044604925e-16 1.0 0.0; origin xyz=0 -0.0225001557729 0.07926 rpy=0 1.30899702752 0 -> xyz=0 -0.0224999 0.07926 rpy=0 1.30899700697 0
- joint r_forearm_mtb_acc_2b7_fixed_joint: origin xyz=-0.11436927713 0.0279967173307 -0.0165298605327 rpy=0.261799479381 0.000370253132778 1.57125811942 -> xyz=-0.114369314675 0.0279969 -0.0165299963729 rpy=0.26179949998 0.000370413042328 1.57125816863
- joint r_forearm_mtb_acc_2b8_fixed_joint: origin xyz=-0.0891879779927 0.00375149154266 0.0348004899258 rpy=0.661159001513 0.147745794174 -0.0919672808581 -> xyz=-0.0891879954459 0.0037515 0.034800424042 rpy=0.661159832193 0.147746087249 -0.0919671195152
- joint r_forearm_mtb_acc_2b9_fixed_joint: origin xyz=-0.0591344983628 0.0504236337681 -0.0187310112996 rpy=-1.76682629734 0.261191812382 0.0540474877723 -> xyz=-0.0591345256166 0.0504239 -0.0187311091679 rpy=-1.76682626732 0.261191225646 0.054048344372
- joint r_shoulder_yaw: axis 0.965925849201 -6.1184868283e-09 -0.258818959594 -> 0.965925843882 -2.22044604925e-16 -0.258818979447; origin xyz=-0.024898847655 2.32747594447e-07 -0.00550748124286 rpy=0 0 0 -> xyz=-0.0253460713232 2.32750427306e-07 -0.00538764806457 rpy=-0.252689546175 0.0085186183214 0.067039889142
- joint r_upper_arm_mtb_acc_2b10_fixed_joint: origin xyz=-0.0412194005144 0.0295878213836 0.0295279 rpy=1.5707969706 1.57078381227 -2.68257108456 -> xyz=-0.0412195 0.029588 0.0295279 rpy=1.57079546365 1.57078381225 -2.68257161164
- joint r_upper_arm_mtb_acc_2b11_fixed_joint: origin xyz=-0.0430565765807 0.0286793709492 0.0760604 rpy=-1.57079619265 -1.57050350759 0.459020791048 -> xyz=-0.0430568 0.02868 0.0760604 rpy=-1.57079614696 -1.57050350741 0.459021725219
- joint r_upper_arm_mtb_acc_2b12_fixed_joint: origin xyz=-0.0430553865107 0.0286807251034 0.0049922 rpy=-1.98902065637 -1.57079632679 0.785398163397 -> xyz=-0.0430555 0.028681 0.0049922 rpy=-1.11177442168 -1.57079632679 0
- joint r_upper_arm_mtb_acc_2b13_fixed_joint: origin xyz=0.010593416831 0.0283497693333 -0.010738 rpy=1.57079632691 -0.000214520111068 2.47803691075 -> xyz=0.010593184 0.02835 -0.010738 rpy=1.57079632702 -0.000214520362041 2.47803674451

Commit message: Sensorised URDF

File: iCubGenova02/iCubGenova02.urdf (robot description, URDF)
Before this commit: robot iCubGenova02, 99 links, 98 joints
Links:
- removed link chest_ems_acc_eb1
- removed link chest_ems_acc_eb2
- removed link chest_ems_acc_eb3
- removed link chest_ems_acc_eb4
- removed link chest_ems_gyro_eb1
- removed link chest_ems_gyro_eb2
- removed link chest_ems_gyro_eb3
- removed link chest_ems_gyro_eb4
- removed link chest_mtb_acc_0b10
- removed link chest_mtb_acc_0b7
- removed link chest_mtb_acc_0b8
- removed link chest_mtb_acc_0b9
- removed link l_forearm_mtb_acc_1b7
- removed link l_forearm_mtb_acc_1b8
- removed link l_forearm_mtb_acc_1b9
- removed link l_lower_leg_ems_acc_eb7
- removed link l_lower_leg_ems_gyro_eb7
- removed link l_lower_leg_mtb_acc_10b10
- removed link l_lower_leg_mtb_acc_10b11
- removed link l_lower_leg_mtb_acc_10b8
- removed link l_lower_leg_mtb_acc_10b9
- removed link l_upper_arm_mtb_acc_1b10
- removed link l_upper_arm_mtb_acc_1b11
- removed link l_upper_arm_mtb_acc_1b12
- removed link l_upper_arm_mtb_acc_1b13
- removed link l_upper_leg_ems_acc_eb10
- removed link l_upper_leg_ems_acc_eb6
- removed link l_upper_leg_ems_gyro_eb10
- removed link l_upper_leg_ems_gyro_eb6
- removed link l_upper_leg_mtb_acc_10b1
- removed link l_upper_leg_mtb_acc_10b2
- removed link l_upper_leg_mtb_acc_10b3
- removed link l_upper_leg_mtb_acc_10b4
- removed link l_upper_leg_mtb_acc_10b5
- removed link l_upper_leg_mtb_acc_10b6
- removed link l_upper_leg_mtb_acc_10b7
- removed link r_foot_mtb_acc_11b12
- removed link r_foot_mtb_acc_11b13
- removed link r_forearm_mtb_acc_2b7
- removed link r_forearm_mtb_acc_2b8
- removed link r_forearm_mtb_acc_2b9
- removed link r_lower_leg_ems_acc_eb9
- removed link r_lower_leg_ems_gyro_eb9
- removed link r_lower_leg_mtb_acc_11b10
- removed link r_lower_leg_mtb_acc_11b11
- removed link r_lower_leg_mtb_acc_11b8
- removed link r_lower_leg_mtb_acc_11b9
- removed link r_upper_arm_mtb_acc_2b10
- removed link r_upper_arm_mtb_acc_2b11
- removed link r_upper_arm_mtb_acc_2b12
- removed link r_upper_arm_mtb_acc_2b13
- removed link r_upper_leg_ems_acc_eb11
- removed link r_upper_leg_ems_acc_eb8
- removed link r_upper_leg_ems_gyro_eb11
- removed link r_upper_leg_ems_gyro_eb8
- removed link r_upper_leg_mtb_acc_11b1
- removed link r_upper_leg_mtb_acc_11b2
- removed link r_upper_leg_mtb_acc_11b3
- removed link r_upper_leg_mtb_acc_11b4
- removed link r_upper_leg_mtb_acc_11b5
- removed link r_upper_leg_mtb_acc_11b6
- removed link r_upper_leg_mtb_acc_11b7
- removed link root_link_ems_acc_eb5
- removed link root_link_ems_gyro_eb5
Joints:
- removed joint chest_ems_acc_eb1_fixed_joint
- removed joint chest_ems_acc_eb2_fixed_joint
- removed joint chest_ems_acc_eb3_fixed_joint
- removed joint chest_ems_acc_eb4_fixed_joint
- removed joint chest_ems_gyro_eb1_fixed_joint
- removed joint chest_ems_gyro_eb2_fixed_joint
- removed joint chest_ems_gyro_eb3_fixed_joint
- removed joint chest_ems_gyro_eb4_fixed_joint
- removed joint chest_mtb_acc_0b10_fixed_joint
- removed joint chest_mtb_acc_0b7_fixed_joint
- removed joint chest_mtb_acc_0b8_fixed_joint
- removed joint chest_mtb_acc_0b9_fixed_joint
- removed joint l_forearm_mtb_acc_1b7_fixed_joint
- removed joint l_forearm_mtb_acc_1b8_fixed_joint
- removed joint l_forearm_mtb_acc_1b9_fixed_joint
- removed joint l_lower_leg_ems_acc_eb7_fixed_joint
- removed joint l_lower_leg_ems_gyro_eb7_fixed_joint
- removed joint l_lower_leg_mtb_acc_10b10_fixed_joint
- removed joint l_lower_leg_mtb_acc_10b11_fixed_joint
- removed joint l_lower_leg_mtb_acc_10b8_fixed_joint
- removed joint l_lower_leg_mtb_acc_10b9_fixed_joint
- removed joint l_upper_arm_mtb_acc_1b10_fixed_joint
- removed joint l_upper_arm_mtb_acc_1b11_fixed_joint
- removed joint l_upper_arm_mtb_acc_1b12_fixed_joint
- removed joint l_upper_arm_mtb_acc_1b13_fixed_joint
- removed joint l_upper_leg_ems_acc_eb10_fixed_joint
- removed joint l_upper_leg_ems_acc_eb6_fixed_joint
- removed joint l_upper_leg_ems_gyro_eb10_fixed_joint
- removed joint l_upper_leg_ems_gyro_eb6_fixed_joint
- removed joint l_upper_leg_mtb_acc_10b1_fixed_joint
- removed joint l_upper_leg_mtb_acc_10b2_fixed_joint
- removed joint l_upper_leg_mtb_acc_10b3_fixed_joint
- removed joint l_upper_leg_mtb_acc_10b4_fixed_joint
- removed joint l_upper_leg_mtb_acc_10b5_fixed_joint
- removed joint l_upper_leg_mtb_acc_10b6_fixed_joint
- removed joint l_upper_leg_mtb_acc_10b7_fixed_joint
- removed joint r_foot_mtb_acc_11b12_fixed_joint
- removed joint r_foot_mtb_acc_11b13_fixed_joint
- removed joint r_forearm_mtb_acc_2b7_fixed_joint
- removed joint r_forearm_mtb_acc_2b8_fixed_joint
- removed joint r_forearm_mtb_acc_2b9_fixed_joint
- removed joint r_lower_leg_ems_acc_eb9_fixed_joint
- removed joint r_lower_leg_ems_gyro_eb9_fixed_joint
- removed joint r_lower_leg_mtb_acc_11b10_fixed_joint
- removed joint r_lower_leg_mtb_acc_11b11_fixed_joint
- removed joint r_lower_leg_mtb_acc_11b8_fixed_joint
- removed joint r_lower_leg_mtb_acc_11b9_fixed_joint
- removed joint r_upper_arm_mtb_acc_2b10_fixed_joint
- removed joint r_upper_arm_mtb_acc_2b11_fixed_joint
- removed joint r_upper_arm_mtb_acc_2b12_fixed_joint
- removed joint r_upper_arm_mtb_acc_2b13_fixed_joint
- removed joint r_upper_leg_ems_acc_eb11_fixed_joint
- removed joint r_upper_leg_ems_acc_eb8_fixed_joint
- removed joint r_upper_leg_ems_gyro_eb11_fixed_joint
- removed joint r_upper_leg_ems_gyro_eb8_fixed_joint
- removed joint r_upper_leg_mtb_acc_11b1_fixed_joint
- removed joint r_upper_leg_mtb_acc_11b2_fixed_joint
- removed joint r_upper_leg_mtb_acc_11b3_fixed_joint
- removed joint r_upper_leg_mtb_acc_11b4_fixed_joint
- removed joint r_upper_leg_mtb_acc_11b5_fixed_joint
- removed joint r_upper_leg_mtb_acc_11b6_fixed_joint
- removed joint r_upper_leg_mtb_acc_11b7_fixed_joint
- removed joint root_link_ems_acc_eb5_fixed_joint
- removed joint root_link_ems_gyro_eb5_fixed_joint
