Commit message: Added IMU and 3 accelerometers on the left leg with respective MTB plugins

File: iCubGenova02/iCubGenova02.urdf (robot description, URDF)
Before this commit: robot iCubGenova02, 102 links, 101 joints
Links:
- removed link chest_ems_acc_eb1
- removed link chest_ems_acc_eb2
- removed link chest_ems_acc_eb3
- removed link chest_ems_acc_eb4
- removed link chest_ems_gyro_eb1
- removed link chest_ems_gyro_eb2
- removed link chest_ems_gyro_eb3
- removed link chest_ems_gyro_eb4
- removed link chest_mtb_acc_0b10
- removed link chest_mtb_acc_0b7
- removed link chest_mtb_acc_0b8
- removed link chest_mtb_acc_0b9
- removed link l_foot_mtb_acc_10b13
- removed link l_forearm_mtb_acc_1b7
- removed link l_forearm_mtb_acc_1b8
- removed link l_forearm_mtb_acc_1b9
- removed link l_lower_leg_ems_acc_eb7
- removed link l_lower_leg_ems_gyro_eb7
- removed link l_lower_leg_mtb_acc_10b10
- removed link l_lower_leg_mtb_acc_10b11
- removed link l_lower_leg_mtb_acc_10b9
- removed link l_upper_arm_mtb_acc_1b10
- removed link l_upper_arm_mtb_acc_1b11
- removed link l_upper_arm_mtb_acc_1b12
- removed link l_upper_arm_mtb_acc_1b13
- removed link l_upper_leg_ems_acc_eb10
- removed link l_upper_leg_ems_acc_eb6
- removed link l_upper_leg_ems_gyro_eb10
- removed link l_upper_leg_ems_gyro_eb6
- removed link l_upper_leg_mtb_acc_10b2
- removed link l_upper_leg_mtb_acc_10b3
- removed link l_upper_leg_mtb_acc_10b4
- removed link l_upper_leg_mtb_acc_10b5
- removed link l_upper_leg_mtb_acc_10b6
- removed link l_upper_leg_mtb_acc_10b7
- removed link r_foot_mtb_acc_11b12
- removed link r_foot_mtb_acc_11b13
- removed link r_forearm_mtb_acc_2b7
- removed link r_forearm_mtb_acc_2b8
- removed link r_forearm_mtb_acc_2b9
- removed link r_lower_leg_ems_acc_eb9
- removed link r_lower_leg_ems_gyro_eb9
- removed link r_lower_leg_mtb_acc_11b10
- removed link r_lower_leg_mtb_acc_11b11
- removed link r_lower_leg_mtb_acc_11b8
- removed link r_lower_leg_mtb_acc_11b9
- removed link r_upper_arm_mtb_acc_2b10
- removed link r_upper_arm_mtb_acc_2b11
- removed link r_upper_arm_mtb_acc_2b12
- removed link r_upper_arm_mtb_acc_2b13
- removed link r_upper_leg_ems_acc_eb11
- removed link r_upper_leg_ems_acc_eb8
- removed link r_upper_leg_ems_gyro_eb11
- removed link r_upper_leg_ems_gyro_eb8
- removed link r_upper_leg_mtb_acc_11b1
- removed link r_upper_leg_mtb_acc_11b2
- removed link r_upper_leg_mtb_acc_11b3
- removed link r_upper_leg_mtb_acc_11b4
- removed link r_upper_leg_mtb_acc_11b5
- removed link r_upper_leg_mtb_acc_11b6
- removed link r_upper_leg_mtb_acc_11b7
- removed link root_link_ems_acc_eb5
- removed link root_link_ems_gyro_eb5
Joints:
- removed joint chest_ems_acc_eb1_fixed_joint
- removed joint chest_ems_acc_eb2_fixed_joint
- removed joint chest_ems_acc_eb3_fixed_joint
- removed joint chest_ems_acc_eb4_fixed_joint
- removed joint chest_ems_gyro_eb1_fixed_joint
- removed joint chest_ems_gyro_eb2_fixed_joint
- removed joint chest_ems_gyro_eb3_fixed_joint
- removed joint chest_ems_gyro_eb4_fixed_joint
- removed joint chest_mtb_acc_0b10_fixed_joint
- removed joint chest_mtb_acc_0b7_fixed_joint
- removed joint chest_mtb_acc_0b8_fixed_joint
- removed joint chest_mtb_acc_0b9_fixed_joint
- removed joint l_foot_mtb_acc_10b13_fixed_joint
- removed joint l_forearm_mtb_acc_1b7_fixed_joint
- removed joint l_forearm_mtb_acc_1b8_fixed_joint
- removed joint l_forearm_mtb_acc_1b9_fixed_joint
- removed joint l_lower_leg_ems_acc_eb7_fixed_joint
- removed joint l_lower_leg_ems_gyro_eb7_fixed_joint
- removed joint l_lower_leg_mtb_acc_10b10_fixed_joint
- removed joint l_lower_leg_mtb_acc_10b11_fixed_joint
- removed joint l_lower_leg_mtb_acc_10b9_fixed_joint
- removed joint l_upper_arm_mtb_acc_1b10_fixed_joint
- removed joint l_upper_arm_mtb_acc_1b11_fixed_joint
- removed joint l_upper_arm_mtb_acc_1b12_fixed_joint
- removed joint l_upper_arm_mtb_acc_1b13_fixed_joint
- removed joint l_upper_leg_ems_acc_eb10_fixed_joint
- removed joint l_upper_leg_ems_acc_eb6_fixed_joint
- removed joint l_upper_leg_ems_gyro_eb10_fixed_joint
- removed joint l_upper_leg_ems_gyro_eb6_fixed_joint
- removed joint l_upper_leg_mtb_acc_10b2_fixed_joint
- removed joint l_upper_leg_mtb_acc_10b3_fixed_joint
- removed joint l_upper_leg_mtb_acc_10b4_fixed_joint
- removed joint l_upper_leg_mtb_acc_10b5_fixed_joint
- removed joint l_upper_leg_mtb_acc_10b6_fixed_joint
- removed joint l_upper_leg_mtb_acc_10b7_fixed_joint
- removed joint r_foot_mtb_acc_11b12_fixed_joint
- removed joint r_foot_mtb_acc_11b13_fixed_joint
- removed joint r_forearm_mtb_acc_2b7_fixed_joint
- removed joint r_forearm_mtb_acc_2b8_fixed_joint
- removed joint r_forearm_mtb_acc_2b9_fixed_joint
- removed joint r_lower_leg_ems_acc_eb9_fixed_joint
- removed joint r_lower_leg_ems_gyro_eb9_fixed_joint
- removed joint r_lower_leg_mtb_acc_11b10_fixed_joint
- removed joint r_lower_leg_mtb_acc_11b11_fixed_joint
- removed joint r_lower_leg_mtb_acc_11b8_fixed_joint
- removed joint r_lower_leg_mtb_acc_11b9_fixed_joint
- removed joint r_upper_arm_mtb_acc_2b10_fixed_joint
- removed joint r_upper_arm_mtb_acc_2b11_fixed_joint
- removed joint r_upper_arm_mtb_acc_2b12_fixed_joint
- removed joint r_upper_arm_mtb_acc_2b13_fixed_joint
- removed joint r_upper_leg_ems_acc_eb11_fixed_joint
- removed joint r_upper_leg_ems_acc_eb8_fixed_joint
- removed joint r_upper_leg_ems_gyro_eb11_fixed_joint
- removed joint r_upper_leg_ems_gyro_eb8_fixed_joint
- removed joint r_upper_leg_mtb_acc_11b1_fixed_joint
- removed joint r_upper_leg_mtb_acc_11b2_fixed_joint
- removed joint r_upper_leg_mtb_acc_11b3_fixed_joint
- removed joint r_upper_leg_mtb_acc_11b4_fixed_joint
- removed joint r_upper_leg_mtb_acc_11b5_fixed_joint
- removed joint r_upper_leg_mtb_acc_11b6_fixed_joint
- removed joint r_upper_leg_mtb_acc_11b7_fixed_joint
- removed joint root_link_ems_acc_eb5_fixed_joint
- removed joint root_link_ems_gyro_eb5_fixed_joint
- joint l_knee: axis -1.0 -0.0 -0.0 -> -1.0 0.0 0.0
- joint r_ankle_roll: axis -0.0 -0.0 -1.0 -> 0.0 0.0 -1.0
- joint r_hip_pitch: axis -1.0 -0.0 -0.0 -> -1.0 0.0 0.0
- joint r_hip_roll: axis -0.0 -0.0 -1.0 -> 0.0 0.0 -1.0

File: iCubGenova02/iCubGenova02NoBattery.urdf (robot description, URDF)
Before this commit: robot iCubGenova02, 102 links, 101 joints
Links:
- removed link imu_frame
- added link imu
Joints:
- removed joint imu_frame_fixed_joint
- added joint imu_fixed_joint: type fixed, parent head, child imu, origin xyz=0.00950000019074 0.133444 0.0093 rpy=-1.57079632679 1.57079632679 0
- joint l_knee: axis -1.0 -0.0 -0.0 -> -1.0 0.0 0.0
- joint r_ankle_roll: axis -0.0 -0.0 -1.0 -> 0.0 0.0 -1.0
- joint r_hip_pitch: axis -1.0 -0.0 -0.0 -> -1.0 0.0 0.0
- joint r_hip_roll: axis -0.0 -0.0 -1.0 -> 0.0 0.0 -1.0

Commit message: Add all left leg MTB sensors Workaround for Gazebo bug on getScopedName()

File: iCubGenova02/iCubGenova02.urdf (robot description, URDF)
Before this commit: robot iCubGenova02, 39 links, 38 joints
Links:
- added link l_foot_mtb_acc_10b13
- added link l_lower_leg_mtb_acc_10b10
- added link l_lower_leg_mtb_acc_10b11
- added link l_lower_leg_mtb_acc_10b9
- added link l_upper_leg_mtb_acc_10b2
- added link l_upper_leg_mtb_acc_10b3
- added link l_upper_leg_mtb_acc_10b4
- added link l_upper_leg_mtb_acc_10b5
- added link l_upper_leg_mtb_acc_10b6
- added link l_upper_leg_mtb_acc_10b7
Joints:
- added joint l_foot_mtb_acc_10b13_fixed_joint: type fixed, parent l_foot, child l_foot_mtb_acc_10b13, origin xyz=0.0805224 0.0118072 -0.001215 rpy=0 0 1.57079632679
- added joint l_lower_leg_mtb_acc_10b10_fixed_joint: type fixed, parent l_lower_leg, child l_lower_leg_mtb_acc_10b10, origin xyz=0.030989 -0.011037 0.05238133 rpy=-1.32645042367 0 1.57079632679
- added joint l_lower_leg_mtb_acc_10b11_fixed_joint: type fixed, parent l_lower_leg, child l_lower_leg_mtb_acc_10b11, origin xyz=-0.0179355 -0.092958 0.0184593 rpy=-1.3089971472 -2.54317885716e-05 1.57078951235
- added joint l_lower_leg_mtb_acc_10b9_fixed_joint: type fixed, parent l_lower_leg, child l_lower_leg_mtb_acc_10b9, origin xyz=0.0665272 -0.043468 0.0259151 rpy=1.30899714594 -0.000112159802878 1.57082638021
- added joint l_upper_leg_mtb_acc_10b2_fixed_joint: type fixed, parent l_upper_leg, child l_upper_leg_mtb_acc_10b2, origin xyz=0.0083839 0.039452 0.05335544 rpy=0.837758036965 -8.62912869137e-05 1.57087402394
- added joint l_upper_leg_mtb_acc_10b3_fixed_joint: type fixed, parent l_upper_leg, child l_upper_leg_mtb_acc_10b3, origin xyz=0.0150706 0.004382 0.053785 rpy=0 0 1.57079632679
- added joint l_upper_leg_mtb_acc_10b4_fixed_joint: type fixed, parent l_upper_leg, child l_upper_leg_mtb_acc_10b4, origin xyz=-0.0144294 0.004382 0.053785 rpy=0 0 1.57079632679
- added joint l_upper_leg_mtb_acc_10b5_fixed_joint: type fixed, parent l_upper_leg, child l_upper_leg_mtb_acc_10b5, origin xyz=-0.0414999 -0.004658 0.03412949 rpy=-1.18682376254 0 1.57079632679
- added joint l_upper_leg_mtb_acc_10b6_fixed_joint: type fixed, parent l_upper_leg, child l_upper_leg_mtb_acc_10b6, origin xyz=0.0178086 -0.026212 -0.043785 rpy=3.14159265359 0 -1.57091243005
- added joint l_upper_leg_mtb_acc_10b7_fixed_joint: type fixed, parent l_upper_leg, child l_upper_leg_mtb_acc_10b7, origin xyz=-0.0141918 -0.026211 -0.043785 rpy=3.14159265359 0 -1.5709453147
