Commit message: Fixed left_hip and right_hip joint limits. Added plugins activating arms inertialMTB sensors. Fixed mtb_acc sensor names in the plugin init config files.

File: icub/icub.urdf (robot description, URDF)
Before this commit: robot iCub, 57 links, 56 joints
Joints:
- joint l_hip_roll: limit lower=-2.07694 upper=0.296706 effort=84 velocity=100 -> lower=0.0 upper=1.57079632679 effort=84 velocity=100
- joint r_hip_roll: limit lower=-2.07694 upper=0.296706 effort=84 velocity=100 -> lower=0.0 upper=1.57079632679 effort=84 velocity=100
